Commit message: Update docs and refactor launch files

File: scout/urdf/scout.urdf (robot description, URDF)
Before this commit: robot scout, 2 links, 1 joints
Joints:
- joint laser_link_joint: origin xyz=0.0 0.0 0.05 rpy=0 0 0 -> xyz=0.17 0.0 0.13 rpy=0 0 0

Commit message: Add localization launch file

File: scout/urdf/scout.urdf (robot description, URDF)
Before this commit: robot scout, 2 links, 1 joints
Joints:
- joint laser_link_joint: origin xyz=0.17 0.0 0.13 rpy=0 0 0 -> xyz=0.17 0.0 0.13 rpy=0 0 3.1416
